Commit message: Edited yaml file to point to the URDF

File: noirbot_description/urdf/noirbot.urdf.xacro (robot description, xacro)
@@ -49,5 +49,5 @@
       <origin xyz="0 -0.015 0" rpy="1.57 0 0" />
       <geometry>
-        <sphere radius="0.072"/>
+        <sphere radius="0.033"/>
       </geometry>
     </collision>

Commit message: Modified MUP axis numbers

File: noirbot_description/urdf/noirbot.urdf.xacro (robot description, xacro)
@@ -111,5 +111,5 @@
   </link>
   <joint name="imu_joint" type="fixed">
-    <origin xyz="0 0 0.0698986241758014" rpy="0 0 0" />
+    <origin xyz="0 0 0.0698986241758014" rpy="3.14159 0 0" />
     <parent link="base_link" />
     <child link="imu_link" />
